Commit message: no hardware

File: legged_examples/legged_unitree/legged_unitree_description/urdf/common/leg.xacro (robot description, xacro)
@@ -33,5 +33,5 @@
                 </xacro:if>
                 <geometry>
-                    <mesh filename="${mesh_path}/hip.dae"
+                    <mesh filename="package://legged_unitree_description/meshes/a1/hip.dae"
                           scale="1 1 1"/>
                 </geometry>
@@ -67,9 +67,9 @@
                 <geometry>
                     <xacro:if value="${mirror_dae == True}">
-                        <mesh filename="${mesh_path}/thigh.dae"
+                        <mesh filename="package://legged_unitree_description/meshes/a1/thigh.dae"
                               scale="1 1 1"/>
                     </xacro:if>
                     <xacro:if value="${mirror_dae == False}">
-                        <mesh filename="${mesh_path}/thigh_mirror.dae"
+                        <mesh filename="package://legged_unitree_description/meshes/a1/thigh_mirror.dae"
                               scale="1 1 1"/>
                     </xacro:if>
@@ -110,5 +110,5 @@
                 <origin rpy="0 0 0" xyz="0 0 0"/>
                 <geometry>
-                    <mesh filename="${mesh_path}/calf.dae"
+                    <mesh filename="package://legged_unitree_description/meshes/a1/calf.dae"
                           scale="1 1 1"/>
                 </geometry>

File: legged_examples/legged_unitree/legged_unitree_description/urdf/robot.xacro (robot description, xacro)
@@ -8,5 +8,5 @@
     <xacro:include filename="$(find legged_unitree_description)/urdf/$(arg robot_type)/const.xacro"/>
 <!--    <xacro:property name="mesh_path" value="../meshes"/>-->
-    <xacro:property name="mesh_path" value="$(find legged_unitree_description)/meshes/$(arg robot_type)"/>
+    <xacro:property name="mesh_path" value="package://legged_unitree_description/meshes/$(arg robot_type)"/>
     <link name="base">
         <visual>
